File: PonchoERG/Aislación.sch (KiCad schematic (older format))
At the start: 9 parts, among them J3 POWER_PONCHO, U7 NCP1117ST33T3G, U8 ADuM6401, U9 ADuM2401

Commit message: Actualización 1.0 - Inclusión de nuevos diodos de protección TPD2E001. - Creación de librería TPD2E001 y rediseño de esquemático. - Reubicación de componentes.
Parts:
- U11: renamed from U8; symbol ADuM6401 -> ADuM6401-RESCUE-PonchoERG
- renumbered U9 to U12, U7 to U13
Changed lines of the file:
@@
 EESchema Schematic File Version 2
+LIBS:PonchoERG-rescue
 LIBS:74xgxx
 LIBS:74xx
@@
 LIBS:PonchoERG
 LIBS:PonchoERG-cache
-LIBS:PonchoERG-rescue
 LIBS:Power
 LIBS:VCC
@@
 $EndDescr
 $Comp
-L ADuM6401 U8
+L ADuM6401-RESCUE-PonchoERG U11
 U 1 1 57C2D878
 P 4600 2200
-F 0 "U8" H 4200 2700 50  0000 L CNN
+AR Path="/57C2D878" Ref="U11"  Part="1"
+AR Path="/57BDC3A8/57C2D878" Ref="U11"  Part="1"
+F 0 "U11" H 4200 2700 50  0000 L CNN
 F 1 "ADuM6401" H 4200 1600 50  0000 L CNN
 F 2 "SMD_Packages:SO-16-W" H 4100 2500 50  0001 C CNN
@@
 	2400 1900 4100 1900
 $Comp
-L NCP1117ST33T3G U7
+L NCP1117ST33T3G U13
 U 1 1 57C39068
 P 2000 1950
-F 0 "U7" H 1800 1750 50  0000 C CNN
+F 0 "U13" H 1800 1750 50  0000 C CNN
 F 1 "NCP1117ST33T3G" H 2000 2150 50  0000 C CNN
 F 2 "TO_SOT_Packages_SMD:SOT-223" H 2000 1950 50  0001 C CNN
@@
 Connection ~ 1400 2600
 $Comp
-L GNDA #PWR023
+L GNDA #PWR024
 U 1 1 57C3B049
 P 2000 2700
-F 0 "#PWR023" H 2000 2450 50  0001 C CNN
+F 0 "#PWR024" H 2000 2450 50  0001 C CNN
 F 1 "GNDA" H 2000 2550 50  0000 C CNN
 F 2 "" H 2000 2700 50  0000 C CNN
@@
 GND_NISO
 $Comp
-L ADuM2401 U9
+L ADuM2401 U12
 U 1 1 57C3167A
 P 4600 4150
-F 0 "U9" H 4300 4650 60  0000 C CNN
+F 0 "U12" H 4300 4650 60  0000 C CNN
 F 1 "ADuM2401" H 4500 3650 60  0000 C CNN
 F 2 "SMD_Packages:SO-16-W" H 4600 4150 60  0001 C CNN
@@
 	6350 4400 6350 3900
 $Comp
-L +5VA #PWR024
+L +5VA #PWR025
 U 1 1 57C3B196
 P 2850 850
-F 0 "#PWR024" H 2850 700 50  0001 C CNN
+F 0 "#PWR025" H 2850 700 50  0001 C CNN
 F 1 "+5VA" H 2850 990 50  0000 C CNN
 F 2 "" H 2850 850 50  0000 C CNN
@@
 $EndComp
 $Comp
-L GNDA #PWR025
+L GNDA #PWR026
 U 1 1 57C3B1B8
 P 2850 1350
-F 0 "#PWR025" H 2850 1100 50  0001 C CNN
+F 0 "#PWR026" H 2850 1100 50  0001 C CNN
 F 1 "GNDA" H 2850 1200 50  0000 C CNN
 F 2 "" H 2850 1350 50  0000 C CNN
@@
 	3800 1800 3800 4400
 $Comp
-L +3.3V #PWR026
+L +3.3V #PWR027
 U 1 1 57C5F657
 P 1400 1800
-F 0 "#PWR026" H 1400 1650 50  0001 C CNN
+F 0 "#PWR027" H 1400 1650 50  0001 C CNN
 F 1 "+3.3V" H 1400 1940 50  0000 C CNN
 F 2 "" H 1400 1800 50  0000 C CNN
@@
 Connection ~ 3800 2500
 $Comp
-L +5VA #PWR027
+L +5VA #PWR028
 U 1 1 57C5F972
 P 3800 1800
-F 0 "#PWR027" H 3800 1650 50  0001 C CNN
+F 0 "#PWR028" H 3800 1650 50  0001 C CNN
 F 1 "+5VA" H 3800 1940 50  0000 C CNN
 F 2 "" H 3800 1800 50  0000 C CNN
@@
 	1600 1900 1400 1900
 $Comp
-L GNDD #PWR028
+L GNDD #PWR029
 U 1 1 57C8A999
 P 1400 2700
-F 0 "#PWR028" H 1400 2450 50  0001 C CNN
+F 0 "#PWR029" H 1400 2450 50  0001 C CNN
 F 1 "GNDD" H 1400 2550 50  0000 C CNN
 F 2 "" H 1400 2700 50  0000 C CNN

Commit message: Reubicación de ADS y componentes pasivos asociados. Sujeto a revisión.
Parts:
- removed NT1: Net_Tie, OtrosFoot:NET-TIE-1mm, symbol Net_Tie
- added R0: 0, Resistors_SMD:R_0805, symbol R
Connections:
- net labels added: +5V
- net labels removed: +5VA
- wire segments 49 -> 51
Changed lines of the file:
@@
 LIBS:ADuM2401
 LIBS:ADuM6401
-LIBS:CKCL44X7R1H
-LIBS:GNDD
 LIBS:NetTie
 LIBS:PonchoERG
 LIBS:PonchoERG-cache
-LIBS:Power
-LIBS:VCC
+LIBS:net-tie
+LIBS:TPD2E001
 EELAYER 25 0
 EELAYER END
@@
 Comment4 ""
 $EndDescr
-$Comp
-L ADuM6401-RESCUE-PonchoERG U11
-U 1 1 57C2D878
-P 4600 2200
-AR Path="/57C2D878" Ref="U11"  Part="1"
-AR Path="/57BDC3A8/57C2D878" Ref="U11"  Part="1"
-F 0 "U11" H 4200 2700 50  0000 L CNN
-F 1 "ADuM6401" H 4200 1600 50  0000 L CNN
-F 2 "SMD_Packages:SO-16-W" H 4100 2500 50  0001 C CNN
-F 3 "" H 4100 2500 50  0000 C CNN
-	1    4600 2200
-	-1   0    0    -1
-$EndComp
 Text HLabel 3300 2400 0    60   Input ~ 0
 MISO
@@
 	2000 2200 2000 2700
 Wire Wire Line
-	1900 2600 4100 2600
+	1850 2600 4100 2600
 Wire Wire Line
 	4100 2000 4000 2000
@@
 	2500 2400 2500 2600
 Connection ~ 2500 2600
-$Comp
-L Net_Tie NT1
-U 1 1 57C3ACEE
-P 1700 2600
-F 0 "NT1" H 1700 2700 60  0000 C CNN
-F 1 "Net_Tie" H 1700 2500 60  0000 C CNN
-F 2 "OtrosFoot:NET-TIE-1mm" H 1700 2600 60  0001 C CNN
-F 3 "" H 1700 2600 60  0000 C CNN
-	1    1700 2600
-	1    0    0    -1
-$EndComp
-Wire Wire Line
-	1500 2600 1400 2600
+Wire Wire Line
+	1400 2600 1550 2600
 Wire Wire Line
 	1400 2400 1400 2700
 Connection ~ 1400 2600
-$Comp
-L GNDA #PWR024
-U 1 1 57C3B049
-P 2000 2700
-F 0 "#PWR024" H 2000 2450 50  0001 C CNN
-F 1 "GNDA" H 2000 2550 50  0000 C CNN
-F 2 "" H 2000 2700 50  0000 C CNN
-F 3 "" H 2000 2700 50  0000 C CNN
-	1    2000 2700
-	1    0    0    -1
-$EndComp
 Text HLabel 5900 2400 2    60   Output ~ 0
 MISO1
@@
 Text Notes 7100 2600 0    60   ~ 0
 GND_NISO
-$Comp
-L ADuM2401 U12
-U 1 1 57C3167A
-P 4600 4150
-F 0 "U12" H 4300 4650 60  0000 C CNN
-F 1 "ADuM2401" H 4500 3650 60  0000 C CNN
-F 2 "SMD_Packages:SO-16-W" H 4600 4150 60  0001 C CNN
-F 3 "" H 4600 4150 60  0000 C CNN
-	1    4600 4150
-	-1   0    0    -1
-$EndComp
 Wire Wire Line
 	5300 3800 5150 3800
@@
 	6350 4400 6350 3900
 $Comp
-L +5VA #PWR025
-U 1 1 57C3B196
-P 2850 850
-F 0 "#PWR025" H 2850 700 50  0001 C CNN
-F 1 "+5VA" H 2850 990 50  0000 C CNN
-F 2 "" H 2850 850 50  0000 C CNN
-F 3 "" H 2850 850 50  0000 C CNN
-	1    2850 850
-	1    0    0    -1
-$EndComp
-$Comp
-L GNDA #PWR026
-U 1 1 57C3B1B8
-P 2850 1350
-F 0 "#PWR026" H 2850 1100 50  0001 C CNN
-F 1 "GNDA" H 2850 1200 50  0000 C CNN
-F 2 "" H 2850 1350 50  0000 C CNN
-F 3 "" H 2850 1350 50  0000 C CNN
-	1    2850 1350
-	1    0    0    -1
-$EndComp
-$Comp
 L C C31
 U 1 1 57C3B1DA
@@
 Wire Wire Line
 	3800 1800 3800 4400
-$Comp
-L +3.3V #PWR027
-U 1 1 57C5F657
-P 1400 1800
-F 0 "#PWR027" H 1400 1650 50  0001 C CNN
-F 1 "+3.3V" H 1400 1940 50  0000 C CNN
-F 2 "" H 1400 1800 50  0000 C CNN
-F 3 "" H 1400 1800 50  0000 C CNN
-	1    1400 1800
-	1    0    0    -1
-$EndComp
 Connection ~ 3800 2500
-$Comp
-L +5VA #PWR028
-U 1 1 57C5F972
-P 3800 1800
-F 0 "#PWR028" H 3800 1650 50  0001 C CNN
-F 1 "+5VA" H 3800 1940 50  0000 C CNN
-F 2 "" H 3800 1800 50  0000 C CNN
-F 3 "" H 3800 1800 50  0000 C CNN
-	1    3800 1800
-	1    0    0    -1
-$EndComp
 Wire Wire Line
 	1600 1900 1400 1900
-$Comp
-L GNDD #PWR029
-U 1 1 57C8A999
-P 1400 2700
-F 0 "#PWR029" H 1400 2450 50  0001 C CNN
-F 1 "GNDD" H 1400 2550 50  0000 C CNN
-F 2 "" H 1400 2700 50  0000 C CNN
-F 3 "" H 1400 2700 50  0000 C CNN
-	1    1400 2700
-	1    0    0    -1
+Wire Wire Line
+	2850 800  2850 850
+Wire Wire Line
+	2850 1350 2850 1450
+Text GLabel 3800 1800 1    60   Input ~ 0
++5V
+Text GLabel 2850 800  1    60   Input ~ 0
++5V
+Text GLabel 1400 1800 1    60   Input ~ 0
++3.3V
+Text GLabel 1400 2700 3    60   Output ~ 0
+GNDD
+Text GLabel 2000 2700 3    60   Output ~ 0
+GNDA
+Text GLabel 2850 1450 3    60   Output ~ 0
+GNDA
+$Comp
+L R R0
+U 1 1 57C7BBDF
+P 1700 2600
+F 0 "R0" V 1600 2550 50  0000 C CNN
+F 1 "0" V 1700 2600 50  0000 C CNN
+F 2 "Resistors_SMD:R_0805" V 1630 2600 50  0001 C CNN
+F 3 "" H 1700 2600 50  0000 C CNN
+	1    1700 2600
+	0    1    1    0
+$EndComp
+$Comp
+L ADuM6401-RESCUE-PonchoERG U11
+U 1 1 57C7EA7C
+P 4600 2200
+AR Path="/57C7EA7C" Ref="U11"  Part="1"
+AR Path="/57BDC3A8/57C7EA7C" Ref="U11"  Part="1"
+F 0 "U11" H 4200 2700 50  0000 L CNN
+F 1 "ADuM6401" H 4200 1600 50  0000 L CNN
+F 2 "SMD_Packages:SO-16-W" H 4100 2500 50  0001 C CNN
+F 3 "" H 4100 2500 50  0000 C CNN
+	1    4600 2200
+	-1   0    0    -1
+$EndComp
+$Comp
+L ADuM2401 U12
+U 1 1 57C7EB57
+P 4600 4150
+F 0 "U12" H 4300 4650 60  0000 C CNN
+F 1 "ADuM2401" H 4500 3650 60  0000 C CNN
+F 2 "SMD_Packages:SO-16-W" H 4600 4150 60  0001 C CNN
+F 3 "" H 4600 4150 60  0000 C CNN
+	1    4600 4150
+	-1   0    0    -1
 $EndComp
 $EndSCHEMATC

Commit message: Subida n.0
Changed lines of the file:
@@
 	4000 2000 4000 2600
 Connection ~ 4000 2600
-Text Notes 3350 1850 0    60   ~ 0
+Text Notes 3500 1250 0    60   ~ 0
 +5V_ISO
 Text Notes 850  1850 0    60   ~ 0
@@
 Wire Notes Line
 	6300 2000 5800 2000
-Text Notes 7100 2500 0    60   ~ 0
+Text Notes 7350 2050 0    60   ~ 0
 +5V_NISO
-Text Notes 7100 2600 0    60   ~ 0
+Text Notes 7050 2750 0    60   ~ 0
 GND_NISO
 Wire Wire Line

Commit message: Última actualización del proyecto. Creación de librería única "PonchoERG.lib" con todos los componentes. Se agregó el conector estilo CIAA para conectar SPI y alimentaciones. Se agregó carpeta con archivos para creación de lista de materiales "PonchoERG.xml" provisoria. Se modificaron todos los pines de alimentación que estaban como etiquetas con los correspondientes. Quedaría solucionar los problemas del ERC respecto a los errores de pines con el famoso PWR_FLAG.
Parts:
- removed J3: POWER_PONCHO, Pin_Headers:Pin_Header_Straight_1x02, symbol CONN_01X02
Connections:
- net +5V_NISO: now reaches U11.1 (VDD1), U11.7 (VDDL), U12.1 (VDD1), U12.7 (VE1)
- net GND_NISO: now reaches U11.2 (GND1), U11.8 (GND1), U12.2 (GND1), U12.8 (GND1)
- net +3.3V renamed +3V3
- net GNDD renamed Earth
Other:
- note removed: "+5V_NISO"
- note removed: "GND_NISO"
Changed lines of the file:
@@
 EESchema Schematic File Version 2
 LIBS:PonchoERG-rescue
-LIBS:74xgxx
-LIBS:74xx
-LIBS:ac-dc
-LIBS:actel
-LIBS:adc-dac
-LIBS:Altera
-LIBS:analog_devices
-LIBS:analog_switches
-LIBS:atmel
-LIBS:audio
-LIBS:brooktre
-LIBS:cmos_ieee
-LIBS:cmos4000
-LIBS:conn
-LIBS:contrib
-LIBS:cypress
-LIBS:dc-dc
-LIBS:device
-LIBS:digital-audio
-LIBS:diode
-LIBS:display
-LIBS:dsp
-LIBS:elec-unifil
-LIBS:ESD_Protection
-LIBS:ftdi
-LIBS:gennum
-LIBS:graphic
-LIBS:hc11
-LIBS:intel
-LIBS:interface
-LIBS:ir
-LIBS:Lattice
-LIBS:linear
-LIBS:logo
-LIBS:maxim
-LIBS:memory
-LIBS:microchip
-LIBS:microchip_dspic33dsc
-LIBS:microchip_pic10mcu
-LIBS:microchip_pic12mcu
-LIBS:microchip_pic16mcu
-LIBS:microchip_pic18mcu
-LIBS:microchip_pic32mcu
-LIBS:microcontrollers
-LIBS:motor_drivers
-LIBS:motorola
-LIBS:msp430
-LIBS:nordicsemi
-LIBS:nxp_armmcu
-LIBS:onsemi
-LIBS:opto
-LIBS:Oscillators
-LIBS:philips
+LIBS:Misc_Poncho_Grande
+LIBS:Poncho_Esqueleto
+LIBS:PonchoERG
 LIBS:power
-LIBS:Power_Management
-LIBS:powerint
-LIBS:pspice
-LIBS:references
-LIBS:regul
-LIBS:relays
-LIBS:rfcom
-LIBS:sensors
-LIBS:silabs
-LIBS:siliconi
-LIBS:stm8
-LIBS:stm32
-LIBS:supertex
-LIBS:switches
-LIBS:texas
-LIBS:transf
-LIBS:transistors
-LIBS:ttl_ieee
-LIBS:valves
-LIBS:video
-LIBS:Xicor
-LIBS:xilinx
-LIBS:Zilog
-LIBS:ADS1299
-LIBS:ADuM2401
-LIBS:ADuM6401
-LIBS:NetTie
-LIBS:PonchoERG
 LIBS:PonchoERG-cache
-LIBS:net-tie
-LIBS:TPD2E001
 EELAYER 25 0
 EELAYER END
@@
 	4000 2000 4000 2600
 Connection ~ 4000 2600
-Text Notes 3500 1250 0    60   ~ 0
+Text Notes 3300 1850 0    60   ~ 0
 +5V_ISO
 Text Notes 850  1850 0    60   ~ 0
@@
 Text Notes 6400 2300 0    60   ~ 0
 SPI to FRDM
-Text Notes 8000 2600 0    60   ~ 0
+Text Notes 7700 2550 0    60   ~ 0
 POWER from FRDM
-$Comp
-L CONN_01X02 J3
-U 1 1 57C3B76D
-P 7800 2550
-F 0 "J3" H 7800 2700 50  0000 C CNN
-F 1 "POWER_PONCHO" V 7900 2550 50  0000 C CNN
-F 2 "Pin_Headers:Pin_Header_Straight_1x02" H 7800 2550 50  0001 C CNN
-F 3 "" H 7800 2550 50  0000 C CNN
-	1    7800 2550
-	1    0    0    -1
-$EndComp
 Wire Notes Line
 	5800 2450 5800 2000
@@
 Wire Notes Line
 	6300 2000 5800 2000
-Text Notes 7350 2050 0    60   ~ 0
-+5V_NISO
-Text Notes 7050 2750 0    60   ~ 0
-GND_NISO
 Wire Wire Line
 	5300 3800 5150 3800
@@
 Wire Wire Line
 	2850 1350 2850 1450
-Text GLabel 3800 1800 1    60   Input ~ 0
-+5V
-Text GLabel 2850 800  1    60   Input ~ 0
-+5V
-Text GLabel 1400 1800 1    60   Input ~ 0
-+3.3V
-Text GLabel 1400 2700 3    60   Output ~ 0
-GNDD
-Text GLabel 2000 2700 3    60   Output ~ 0
-GNDA
-Text GLabel 2850 1450 3    60   Output ~ 0
-GNDA
 $Comp
 L R R0
@@
 	-1   0    0    -1
 $EndComp
+$Comp
+L GNDA-RESCUE-PonchoERG #PWR031
+U 1 1 57CB14DA
+P 2000 2700
+F 0 "#PWR031" H 2000 2450 50  0001 C CNN
+F 1 "GNDA" H 2000 2550 50  0000 C CNN
+F 2 "" H 2000 2700 50  0000 C CNN
+F 3 "" H 2000 2700 50  0000 C CNN
+	1    2000 2700
+	1    0    0    -1
+$EndComp
+$Comp
+L GNDA-RESCUE-PonchoERG #PWR032
+U 1 1 57CB1500
+P 2850 1450
+F 0 "#PWR032" H 2850 1200 50  0001 C CNN
+F 1 "GNDA" H 2850 1300 50  0000 C CNN
+F 2 "" H 2850 1450 50  0000 C CNN
+F 3 "" H 2850 1450 50  0000 C CNN
+	1    2850 1450
+	1    0    0    -1
+$EndComp
+$Comp
+L Earth #PWR033
+U 1 1 57CB1526
+P 1400 2700
+F 0 "#PWR033" H 1400 2450 50  0001 C CNN
+F 1 "Earth" H 1400 2550 50  0001 C CNN
+F 2 "" H 1400 2700 50  0000 C CNN
+F 3 "" H 1400 2700 50  0000 C CNN
+	1    1400 2700
+	1    0    0    -1
+$EndComp
+$Comp
+L +3.3V-RESCUE-PonchoERG #PWR?
+U 1 1 57CB154C
+P 1400 1800
+AR Path="/57CB154C" Ref="#PWR?"  Part="1"
+AR Path="/57BDC3A8/57CB154C" Ref="#PWR034"  Part="1"
+F 0 "#PWR034" H 1400 1650 50  0001 C CNN
+F 1 "+3.3V" H 1400 1940 50  0000 C CNN
+F 2 "" H 1400 1800 50  0000 C CNN
+F 3 "" H 1400 1800 50  0000 C CNN
+	1    1400 1800
+	1    0    0    -1
+$EndComp
+$Comp
+L +5V #PWR035
+U 1 1 57CB1572
+P 2850 800
+F 0 "#PWR035" H 2850 650 50  0001 C CNN
+F 1 "+5V" H 2850 940 50  0000 C CNN
+F 2 "" H 2850 800 50  0000 C CNN
+F 3 "" H 2850 800 50  0000 C CNN
+	1    2850 800
+	1    0    0    -1
+$EndComp
+$Comp
+L +5V #PWR036
+U 1 1 57CB1598
+P 3800 1800
+F 0 "#PWR036" H 3800 1650 50  0001 C CNN
+F 1 "+5V" H 3800 1940 50  0000 C CNN
+F 2 "" H 3800 1800 50  0000 C CNN
+F 3 "" H 3800 1800 50  0000 C CNN
+	1    3800 1800
+	1    0    0    -1
+$EndComp
+Text Label 7600 2500 2    60   ~ 0
++5V_NISO
+Text Label 7600 2600 2    60   ~ 0
+GND_NISO
+Wire Notes Line
+	7100 2400 7100 2650
+Wire Notes Line
+	7100 2650 7650 2650
+Wire Notes Line
+	7650 2650 7650 2400
+Wire Notes Line
+	7650 2400 7100 2400
 $EndSCHEMATC

Commit message: Inclusión en esquemáticos de los nuevos bloques de circuitos para la utilización de las líneas del BIAS. Actualización de librería de proyecto. Objetivo de este comit: revisar actualización e inclusión de BIAS.
Connections:
- net PWDN/: now reaches U12.12 (VOC)
- net PWDN/1: now reaches U12.5 (VIC)
- no-connect marks 2 -> 0
Changed lines of the file:
@@
 LIBS:PonchoERG
 LIBS:power
+LIBS:74xgxx
+LIBS:74xx
+LIBS:ac-dc
+LIBS:actel
+LIBS:adc-dac
+LIBS:Altera
+LIBS:analog_devices
+LIBS:analog_switches
+LIBS:atmel
+LIBS:audio
+LIBS:brooktre
+LIBS:cmos_ieee
+LIBS:cmos4000
+LIBS:conn
+LIBS:contrib
+LIBS:cypress
+LIBS:dc-dc
+LIBS:device
+LIBS:digital-audio
+LIBS:diode
+LIBS:display
+LIBS:dsp
+LIBS:elec-unifil
+LIBS:ESD_Protection
+LIBS:ftdi
+LIBS:gennum
+LIBS:graphic
+LIBS:hc11
+LIBS:intel
+LIBS:interface
+LIBS:ir
+LIBS:Lattice
+LIBS:linear
+LIBS:logo
+LIBS:maxim
+LIBS:memory
+LIBS:microchip
+LIBS:microchip_dspic33dsc
+LIBS:microchip_pic10mcu
+LIBS:microchip_pic12mcu
+LIBS:microchip_pic16mcu
+LIBS:microchip_pic18mcu
+LIBS:microchip_pic32mcu
+LIBS:microcontrollers
+LIBS:motor_drivers
+LIBS:motorola
+LIBS:msp430
+LIBS:nordicsemi
+LIBS:nxp_armmcu
+LIBS:onsemi
+LIBS:opto
+LIBS:Oscillators
+LIBS:philips
+LIBS:Power_Management
+LIBS:powerint
+LIBS:pspice
+LIBS:references
+LIBS:regul
+LIBS:relays
+LIBS:rfcom
+LIBS:sensors
+LIBS:silabs
+LIBS:siliconi
+LIBS:stm8
+LIBS:stm32
+LIBS:supertex
+LIBS:switches
+LIBS:texas
+LIBS:transf
+LIBS:transistors
+LIBS:ttl_ieee
+LIBS:valves
+LIBS:video
+LIBS:Xicor
+LIBS:xilinx
+LIBS:Zilog
 LIBS:PonchoERG-cache
 EELAYER 25 0
@@
 Text HLabel 5900 4300 2    60   Output ~ 0
 DRDY/1
-NoConn ~ 5150 4200
-NoConn ~ 4050 4200
 Wire Wire Line
 	5150 4000 5900 4000
@@
 Wire Notes Line
 	7650 2400 7100 2400
+Text HLabel 5900 4200 2    60   Input ~ 0
+PWDN/1
+Text HLabel 3300 4200 0    60   Output ~ 0
+PWDN/
+Wire Wire Line
+	3300 4200 4050 4200
+Wire Wire Line
+	5150 4200 5900 4200
 $EndSCHEMATC
