File: Desarrollo/Hardware/ADS1299.sch (KiCad schematic (older format))
At the start: 30 parts, among them J2 I/O's Multi Propósito, U10 ADS1299, U14 OPA2376_NI

Commit message: Finalización de primer ruteo estimado. Revisión de cantidad de v
Parts:
- added JP5: -AVSS, Pin_Headers:Pin_Header_Straight_1x03, symbol JUMPER3
Connections:
- net GNDA: now also JP5.3; no longer C37.1, C40.1, U14.4 (V-), U14.4 (V-)
- new net: C37.1, C40.1, JP5.2, U14.4 (V-), U14.4 (V-)
- no-connect marks 4 -> 5
Changed lines of the file:
@@
 encoding utf-8
 Sheet 3 4
-Title ""
+Title "ADS1299"
 Date ""
-Rev ""
-Comp ""
+Rev "1.0"
+Comp "Bruno Javier Cesario"
 Comment1 ""
 Comment2 ""
@@
 P 7050 3800
 AR Path="/57CB1828" Ref="#PWR?"  Part="1"
-AR Path="/57BDC369/57CB1828" Ref="#PWR09"  Part="1"
-F 0 "#PWR09" H 7050 3650 50  0001 C CNN
+AR Path="/57BDC369/57CB1828" Ref="#PWR010"  Part="1"
+F 0 "#PWR010" H 7050 3650 50  0001 C CNN
 F 1 "+3.3V" H 7050 3940 50  0000 C CNN
 F 2 "" H 7050 3800 50  0000 C CNN
@@
 P 9000 2400
 AR Path="/57CB18B2" Ref="#PWR?"  Part="1"
-AR Path="/57BDC369/57CB18B2" Ref="#PWR010"  Part="1"
-F 0 "#PWR010" H 9000 2250 50  0001 C CNN
+AR Path="/57BDC369/57CB18B2" Ref="#PWR011"  Part="1"
+F 0 "#PWR011" H 9000 2250 50  0001 C CNN
 F 1 "+3.3V" H 9000 2540 50  0000 C CNN
 F 2 "" H 9000 2400 50  0000 C CNN
@@
 $EndComp
 $Comp
-L +5V #PWR011
+L +5V #PWR012
 U 1 1 57CB18ED
 P 9900 2400
-F 0 "#PWR011" H 9900 2250 50  0001 C CNN
+F 0 "#PWR012" H 9900 2250 50  0001 C CNN
 F 1 "+5V" H 9900 2540 50  0000 C CNN
 F 2 "" H 9900 2400 50  0000 C CNN
@@
 $EndComp
 $Comp
-L Earth #PWR012
+L Earth #PWR013
 U 1 1 57CB195C
 P 4500 5600
-F 0 "#PWR012" H 4500 5350 50  0001 C CNN
+F 0 "#PWR013" H 4500 5350 50  0001 C CNN
 F 1 "Earth" H 4500 5450 50  0001 C CNN
 F 2 "" H 4500 5600 50  0000 C CNN
@@
 $EndComp
 $Comp
-L Earth #PWR013
+L Earth #PWR014
 U 1 1 57CB198A
 P 6500 5500
-F 0 "#PWR013" H 6500 5250 50  0001 C CNN
+F 0 "#PWR014" H 6500 5250 50  0001 C CNN
 F 1 "Earth" H 6500 5350 50  0001 C CNN
 F 2 "" H 6500 5500 50  0000 C CNN
@@
 $EndComp
 $Comp
-L Earth #PWR014
+L Earth #PWR015
 U 1 1 57CB19B8
 P 7200 4500
-F 0 "#PWR014" H 7200 4250 50  0001 C CNN
+F 0 "#PWR015" H 7200 4250 50  0001 C CNN
 F 1 "Earth" H 7200 4350 50  0001 C CNN
 F 2 "" H 7200 4500 50  0000 C CNN
@@
 $EndComp
 $Comp
-L Earth #PWR015
+L Earth #PWR016
 U 1 1 57CB19E6
 P 6650 3500
-F 0 "#PWR015" H 6650 3250 50  0001 C CNN
+F 0 "#PWR016" H 6650 3250 50  0001 C CNN
 F 1 "Earth" H 6650 3350 50  0001 C CNN
 F 2 "" H 6650 3500 50  0000 C CNN
@@
 $EndComp
 $Comp
-L Earth #PWR016
+L Earth #PWR017
 U 1 1 57CB1A14
 P 9000 3100
-F 0 "#PWR016" H 9000 2850 50  0001 C CNN
+F 0 "#PWR017" H 9000 2850 50  0001 C CNN
 F 1 "Earth" H 9000 2950 50  0001 C CNN
 F 2 "" H 9000 3100 50  0000 C CNN
@@
 $EndComp
 $Comp
-L GNDA-RESCUE-PonchoERG #PWR017
+L GNDA-RESCUE-PonchoERG #PWR018
 U 1 1 57CB1A83
 P 7400 2700
-F 0 "#PWR017" H 7400 2450 50  0001 C CNN
+F 0 "#PWR018" H 7400 2450 50  0001 C CNN
 F 1 "GNDA" H 7400 2550 50  0000 C CNN
 F 2 "" H 7400 2700 50  0000 C CNN
@@
 $EndComp
 $Comp
-L GNDA-RESCUE-PonchoERG #PWR018
+L GNDA-RESCUE-PonchoERG #PWR019
 U 1 1 57CB1AB1
 P 9900 3100
-F 0 "#PWR018" H 9900 2850 50  0001 C CNN
+F 0 "#PWR019" H 9900 2850 50  0001 C CNN
 F 1 "GNDA" H 9900 2950 50  0000 C CNN
 F 2 "" H 9900 3100 50  0000 C CNN
@@
 $EndComp
 $Comp
-L GNDA-RESCUE-PonchoERG #PWR019
+L GNDA-RESCUE-PonchoERG #PWR020
 U 1 1 57CB1ADF
 P 3500 4200
-F 0 "#PWR019" H 3500 3950 50  0001 C CNN
+F 0 "#PWR020" H 3500 3950 50  0001 C CNN
 F 1 "GNDA" H 3500 4050 50  0000 C CNN
 F 2 "" H 3500 4200 50  0000 C CNN
@@
 $EndComp
 $Comp
-L GNDA-RESCUE-PonchoERG #PWR020
+L GNDA-RESCUE-PonchoERG #PWR021
 U 1 1 57CB1B0D
 P 3600 5600
-F 0 "#PWR020" H 3600 5350 50  0001 C CNN
+F 0 "#PWR021" H 3600 5350 50  0001 C CNN
 F 1 "GNDA" H 3600 5450 50  0000 C CNN
 F 2 "" H 3600 5600 50  0000 C CNN
@@
 $EndComp
 $Comp
-L GNDA-RESCUE-PonchoERG #PWR021
+L GNDA-RESCUE-PonchoERG #PWR022
 U 1 1 57CB1B3B
 P 7750 3700
-F 0 "#PWR021" H 7750 3450 50  0001 C CNN
+F 0 "#PWR022" H 7750 3450 50  0001 C CNN
 F 1 "GNDA" H 7750 3550 50  0000 C CNN
 F 2 "" H 7750 3700 50  0000 C CNN
@@
 $EndComp
 $Comp
-L +5V #PWR022
+L +5V #PWR023
 U 1 1 57CB3AA5
 P 7100 2600
-F 0 "#PWR022" H 7100 2450 50  0001 C CNN
+F 0 "#PWR023" H 7100 2450 50  0001 C CNN
 F 1 "+5V" H 7100 2740 50  0000 C CNN
 F 2 "" H 7100 2600 50  0000 C CNN
@@
 $EndComp
 $Comp
-L +5V #PWR023
+L +5V #PWR024
 U 1 1 57CB3AD3
 P 3700 3700
-F 0 "#PWR023" H 3700 3550 50  0001 C CNN
+F 0 "#PWR024" H 3700 3550 50  0001 C CNN
 F 1 "+5V" H 3700 3840 50  0000 C CNN
 F 2 "" H 3700 3700 50  0000 C CNN
@@
 	4550 1550 6250 1550
 Connection ~ 3600 750
-$Comp
-L GNDA-RESCUE-PonchoERG #PWR024
-U 1 1 57CCF983
-P 3600 1900
-F 0 "#PWR024" H 3600 1650 50  0001 C CNN
-F 1 "GNDA" H 3600 1750 50  0000 C CNN
-F 2 "" H 3600 1900 50  0000 C CNN
-F 3 "" H 3600 1900 50  0000 C CNN
-	1    3600 1900
-	1    0    0    -1
-$EndComp
 Connection ~ 3600 1750
 $Comp
@@
 	1    0    0    -1
 $EndComp
-Wire Wire Line
-	3600 1550 3600 1900
 $Comp
 L GNDA-RESCUE-PonchoERG #PWR028
@@
 $EndComp
 Wire Wire Line
-	1500 4750 1650 4750
+	1500 4750 2600 4750
+Connection ~ 1650 4750
 $Comp
 L GNDA-RESCUE-PonchoERG #PWR031
-U 1 1 57CDA7F0
-P 1650 4900
-F 0 "#PWR031" H 1650 4650 50  0001 C CNN
-F 1 "GNDA" H 1650 4750 50  0000 C CNN
-F 2 "" H 1650 4900 50  0000 C CNN
-F 3 "" H 1650 4900 50  0000 C CNN
-	1    1650 4900
-	1    0    0    -1
-$EndComp
-Connection ~ 1650 4750
-$Comp
-L GNDA-RESCUE-PonchoERG #PWR032
 U 1 1 57CDA7F7
-P 1100 4850
-F 0 "#PWR032" H 1100 4600 50  0001 C CNN
-F 1 "GNDA" H 1100 4700 50  0000 C CNN
-F 2 "" H 1100 4850 50  0000 C CNN
-F 3 "" H 1100 4850 50  0000 C CNN
-	1    1100 4850
-	1    0    0    -1
-$EndComp
-Wire Wire Line
-	1100 4850 1100 4750
-Wire Wire Line
-	1100 4750 1200 4750
-Wire Wire Line
-	1650 4550 1650 4900
+P 950 4900
+F 0 "#PWR031" H 950 4650 50  0001 C CNN
+F 1 "GNDA" H 950 4750 50  0000 C CNN
+F 2 "" H 950 4900 50  0000 C CNN
+F 3 "" H 950 4900 50  0000 C CNN
+	1    950  4900
+	1    0    0    -1
+$EndComp
+Wire Wire Line
+	1650 4550 1650 5400
 Wire Wire Line
 	1250 1500 1400 1500
@@
 Text Notes 9700 900  0    60   ~ 0
 Nota:\n\nNI: Not Installed
+Wire Wire Line
+	2600 4750 2600 2200
+Wire Wire Line
+	2600 2200 3600 2200
+Wire Wire Line
+	3600 2200 3600 1550
+Wire Wire Line
+	950  4900 950  4750
+Wire Wire Line
+	950  4750 1200 4750
+$Comp
+L JUMPER3 JP5
+U 1 1 57CFEB0F
+P 1650 5500
+F 0 "JP5" H 1700 5400 50  0000 L CNN
+F 1 "-AVSS" H 1650 5600 50  0000 C BNN
+F 2 "Pin_Headers:Pin_Header_Straight_1x03" H 1650 5500 50  0001 C CNN
+F 3 "" H 1650 5500 50  0000 C CNN
+	1    1650 5500
+	-1   0    0    1
+$EndComp
+Wire Wire Line
+	1400 5500 1150 5500
+Wire Wire Line
+	1150 5500 1150 4750
+Connection ~ 1150 4750
+NoConn ~ 1900 5500
 $EndSCHEMATC

Commit message: Última actualización de ruteo. Redimensión de placa. Cambio de ancho de algunas pistas. Cambio de componentes. Agregado de inductancias de aislación de masas y alimentación +5V.
Parts:
- C39, C40: value NI -> 1uF
- R20: value 392k -> 390k
Connections:
- net GNDA: now also U10.60 (BIASREF)
Changed lines of the file:
@@
 	6400 2900 6600 2900
 Wire Wire Line
-	6600 2800 6600 3300
+	6600 2600 6600 3300
 Connection ~ 6600 2800
 Wire Wire Line
@@
 P 6000 1800
 F 0 "R20" H 6050 1900 50  0000 L CNN
-F 1 "392k" H 6050 1700 50  0000 L CNN
+F 1 "390k" H 6050 1700 50  0000 L CNN
 F 2 "Resistors_SMD:R_0805" H 6000 1800 50  0001 C CNN
 F 3 "" H 6000 1800 50  0000 C CNN
@@
 P 1350 3750
 F 0 "C39" H 1150 3850 50  0000 L CNN
-F 1 "NI" H 1250 3650 50  0000 L CNN
+F 1 "1uF" H 1150 3650 50  0000 L CNN
 F 2 "Capacitors_SMD:C_0805" H 1388 3600 50  0001 C CNN
 F 3 "" H 1350 3750 50  0000 C CNN
@@
 P 1350 4750
 F 0 "C40" H 1450 4850 50  0000 L CNN
-F 1 "NI" H 1450 4650 50  0000 L CNN
+F 1 "1uF" H 1450 4650 50  0000 L CNN
 F 2 "Capacitors_SMD:C_0805" H 1388 4600 50  0001 C CNN
 F 3 "" H 1350 4750 50  0000 C CNN
@@
 Connection ~ 1150 4750
 NoConn ~ 1900 5500
+Wire Wire Line
+	6400 2600 6600 2600
 $EndSCHEMATC
