File: Desarrollo/Hardware/Aislación.sch (KiCad schematic (older format))
At the start: 13 parts, among them U11 ADuM6401, U12 ADuM2401, U13 NCP1117ST33T3G

Commit message: Actualización final con todas las revisiones corregidas. Realizar revisión FINAL.
Parts:
- added FD1, FD2, FD3, FD4, FD5, FD6, FD7, FD8, FD9: Fiducial, Fiducials:Fiducial_1mm_Dia_2.54mm_Outer_CopperTop, symbol Fiducial
- added MH1, MH2, MH3, MH4: PCB_HOLE, Connect:1pin, symbol PCB_HOLE
Connections:
- net GNDA: now also MH1.1, MH2.1
- net GND_NISO: now also MH3.1, MH4.1
Other:
- note added: "ADS1299"
- note added: "Bottom"
- note added: "Fiduciales"
- note added: "Orificios de Montaje"
- note added: "Top"
Changed lines of the file:
@@
 $EndComp
 $Comp
-L GNDA-RESCUE-PonchoERG #PWR031
+L GNDA-RESCUE-PonchoERG #PWR032
 U 1 1 57CB14DA
 P 2000 2700
-F 0 "#PWR031" H 2000 2450 50  0001 C CNN
+F 0 "#PWR032" H 2000 2450 50  0001 C CNN
 F 1 "GNDA" H 2000 2550 50  0000 C CNN
 F 2 "" H 2000 2700 50  0000 C CNN
@@
 $EndComp
 $Comp
-L GNDA-RESCUE-PonchoERG #PWR032
+L GNDA-RESCUE-PonchoERG #PWR033
 U 1 1 57CB1500
 P 2850 1450
-F 0 "#PWR032" H 2850 1200 50  0001 C CNN
+F 0 "#PWR033" H 2850 1200 50  0001 C CNN
 F 1 "GNDA" H 2850 1300 50  0000 C CNN
 F 2 "" H 2850 1450 50  0000 C CNN
@@
 $EndComp
 $Comp
-L DGND #PWR033
+L DGND #PWR034
 U 1 1 57CB1526
 P 1050 2700
-F 0 "#PWR033" H 1050 2450 50  0001 C CNN
+F 0 "#PWR034" H 1050 2450 50  0001 C CNN
 F 1 "DGND" H 1050 2550 50  0001 C CNN
 F 2 "" H 1050 2700 50  0000 C CNN
@@
 P 1050 1800
 AR Path="/57CB154C" Ref="#PWR?"  Part="1"
-AR Path="/57BDC3A8/57CB154C" Ref="#PWR034"  Part="1"
-F 0 "#PWR034" H 1050 1650 50  0001 C CNN
+AR Path="/57BDC3A8/57CB154C" Ref="#PWR035"  Part="1"
+F 0 "#PWR035" H 1050 1650 50  0001 C CNN
 F 1 "+3.3V" H 1050 1940 50  0000 C CNN
 F 2 "" H 1050 1800 50  0000 C CNN
@@
 $EndComp
 $Comp
-L +5V #PWR035
+L +5V #PWR036
 U 1 1 57CB1572
 P 2850 800
-F 0 "#PWR035" H 2850 650 50  0001 C CNN
+F 0 "#PWR036" H 2850 650 50  0001 C CNN
 F 1 "+5V" H 2850 940 50  0000 C CNN
 F 2 "" H 2850 800 50  0000 C CNN
@@
 $EndComp
 $Comp
-L +5V #PWR036
+L +5V #PWR037
 U 1 1 57CB1598
 P 3800 1800
-F 0 "#PWR036" H 3800 1650 50  0001 C CNN
+F 0 "#PWR037" H 3800 1650 50  0001 C CNN
 F 1 "+5V" H 3800 1940 50  0000 C CNN
 F 2 "" H 3800 1800 50  0000 C CNN
@@
 	5650 3650 5400 3650
 Connection ~ 5400 3650
+$Comp
+L Fiducial FD1
+U 1 1 580D56F9
+P 9200 4900
+F 0 "FD1" H 9200 5100 60  0000 C CNN
+F 1 "Fiducial" H 9200 4700 60  0000 C CNN
+F 2 "Fiducials:Fiducial_1mm_Dia_2.54mm_Outer_CopperTop" H 9200 4900 60  0001 C CNN
+F 3 "" H 9200 4900 60  0000 C CNN
+	1    9200 4900
+	1    0    0    -1
+$EndComp
+$Comp
+L Fiducial FD2
+U 1 1 580D57A0
+P 9700 4900
+F 0 "FD2" H 9700 5100 60  0000 C CNN
+F 1 "Fiducial" H 9700 4700 60  0000 C CNN
+F 2 "Fiducials:Fiducial_1mm_Dia_2.54mm_Outer_CopperTop" H 9700 4900 60  0001 C CNN
+F 3 "" H 9700 4900 60  0000 C CNN
+	1    9700 4900
+	1    0    0    -1
+$EndComp
+$Comp
+L Fiducial FD3
+U 1 1 580D57EB
+P 10200 4900
+F 0 "FD3" H 10200 5100 60  0000 C CNN
+F 1 "Fiducial" H 10200 4700 60  0000 C CNN
+F 2 "Fiducials:Fiducial_1mm_Dia_2.54mm_Outer_CopperTop" H 10200 4900 60  0001 C CNN
+F 3 "" H 10200 4900 60  0000 C CNN
+	1    10200 4900
+	1    0    0    -1
+$EndComp
+$Comp
+L Fiducial FD4
+U 1 1 580D583B
+P 10700 4900
+F 0 "FD4" H 10700 5100 60  0000 C CNN
+F 1 "Fiducial" H 10700 4700 60  0000 C CNN
+F 2 "Fiducials:Fiducial_1mm_Dia_2.54mm_Outer_CopperTop" H 10700 4900 60  0001 C CNN
+F 3 "" H 10700 4900 60  0000 C CNN
+	1    10700 4900
+	1    0    0    -1
+$EndComp
+Text Notes 9750 4550 0    60   ~ 12
+Fiduciales
+$Comp
+L PCB_HOLE MH2
+U 1 1 580D7138
+P 7050 5550
+F 0 "MH2" H 7000 5700 60  0000 C CNN
+F 1 "PCB_HOLE" H 7050 5450 60  0001 C CNN
+F 2 "Connect:1pin" H 6900 5600 60  0001 C CNN
+F 3 "PCB HOLE" H 7000 5700 60  0001 C CNN
+	1    7050 5550
+	1    0    0    -1
+$EndComp
+$Comp
+L PCB_HOLE MH3
+U 1 1 580D719D
+P 7550 5550
+F 0 "MH3" H 7500 5700 60  0000 C CNN
+F 1 "PCB_HOLE" H 7550 5450 60  0001 C CNN
+F 2 "Connect:1pin" H 7400 5600 60  0001 C CNN
+F 3 "PCB HOLE" H 7500 5700 60  0001 C CNN
+	1    7550 5550
+	1    0    0    -1
+$EndComp
+$Comp
+L PCB_HOLE MH4
+U 1 1 580D71F6
+P 8050 5550
+F 0 "MH4" H 8000 5700 60  0000 C CNN
+F 1 "PCB_HOLE" H 8050 5450 60  0001 C CNN
+F 2 "Connect:1pin" H 7900 5600 60  0001 C CNN
+F 3 "PCB HOLE" H 8000 5700 60  0001 C CNN
+	1    8050 5550
+	1    0    0    -1
+$EndComp
+$Comp
+L PCB_HOLE MH1
+U 1 1 580D724E
+P 6550 5550
+F 0 "MH1" H 6500 5700 60  0000 C CNN
+F 1 "PCB_HOLE" H 6550 5450 60  0001 C CNN
+F 2 "Connect:1pin" H 6400 5600 60  0001 C CNN
+F 3 "PCB HOLE" H 6500 5700 60  0001 C CNN
+	1    6550 5550
+	1    0    0    -1
+$EndComp
+$Comp
+L GNDA #PWR038
+U 1 1 580D729E
+P 6800 6100
+F 0 "#PWR038" H 6800 6100 40  0001 C CNN
+F 1 "GNDA" H 6800 6030 40  0000 C CNN
+F 2 "" H 6800 6100 60  0000 C CNN
+F 3 "" H 6800 6100 60  0000 C CNN
+	1    6800 6100
+	1    0    0    -1
+$EndComp
+Wire Wire Line
+	6800 6100 6800 5950
+Wire Wire Line
+	6550 5950 7050 5950
+Wire Wire Line
+	6550 5950 6550 5550
+Wire Wire Line
+	7050 5950 7050 5550
+Connection ~ 6800 5950
+Wire Wire Line
+	7550 5550 7550 5950
+Wire Wire Line
+	7550 5950 8050 5950
+Wire Wire Line
+	8050 5950 8050 5550
+Wire Wire Line
+	7800 6100 7800 5950
+Connection ~ 7800 5950
+$Comp
+L Fiducial FD9
+U 1 1 580D7BB1
+P 9950 6200
+F 0 "FD9" H 9950 6400 60  0000 C CNN
+F 1 "Fiducial" H 9950 6000 60  0000 C CNN
+F 2 "Fiducials:Fiducial_1mm_Dia_2.54mm_Outer_CopperTop" H 9950 6200 60  0001 C CNN
+F 3 "" H 9950 6200 60  0000 C CNN
+	1    9950 6200
+	1    0    0    -1
+$EndComp
+$Comp
+L Fiducial FD5
+U 1 1 580D9264
+P 9200 5550
+F 0 "FD5" H 9200 5750 60  0000 C CNN
+F 1 "Fiducial" H 9200 5350 60  0000 C CNN
+F 2 "Fiducials:Fiducial_1mm_Dia_2.54mm_Outer_CopperTop" H 9200 5550 60  0001 C CNN
+F 3 "" H 9200 5550 60  0000 C CNN
+	1    9200 5550
+	1    0    0    -1
+$EndComp
+$Comp
+L Fiducial FD6
+U 1 1 580D926B
+P 9700 5550
+F 0 "FD6" H 9700 5750 60  0000 C CNN
+F 1 "Fiducial" H 9700 5350 60  0000 C CNN
+F 2 "Fiducials:Fiducial_1mm_Dia_2.54mm_Outer_CopperTop" H 9700 5550 60  0001 C CNN
+F 3 "" H 9700 5550 60  0000 C CNN
+	1    9700 5550
+	1    0    0    -1
+$EndComp
+$Comp
+L Fiducial FD7
+U 1 1 580D9272
+P 10200 5550
+F 0 "FD7" H 10200 5750 60  0000 C CNN
+F 1 "Fiducial" H 10200 5350 60  0000 C CNN
+F 2 "Fiducials:Fiducial_1mm_Dia_2.54mm_Outer_CopperTop" H 10200 5550 60  0001 C CNN
+F 3 "" H 10200 5550 60  0000 C CNN
+	1    10200 5550
+	1    0    0    -1
+$EndComp
+$Comp
+L Fiducial FD8
+U 1 1 580D9279
+P 10700 5550
+F 0 "FD8" H 10700 5750 60  0000 C CNN
+F 1 "Fiducial" H 10700 5350 60  0000 C CNN
+F 2 "Fiducials:Fiducial_1mm_Dia_2.54mm_Outer_CopperTop" H 10700 5550 60  0001 C CNN
+F 3 "" H 10700 5550 60  0000 C CNN
+	1    10700 5550
+	1    0    0    -1
+$EndComp
+Text Notes 6800 5200 0    60   ~ 12
+Orificios de Montaje
+Wire Notes Line
+	9000 4600 10900 4600
+Wire Notes Line
+	10900 4600 10900 5900
+Wire Notes Line
+	10900 5900 9000 5900
+Wire Notes Line
+	9000 5900 9000 4600
+Wire Notes Line
+	9000 5250 10900 5250
+Wire Notes Line
+	9650 5900 9650 6450
+Wire Notes Line
+	9650 6450 10250 6450
+Wire Notes Line
+	10250 6450 10250 5900
+Text Notes 8750 4950 0    60   ~ 12
+Top
+Text Notes 8600 5600 0    60   ~ 12
+Bottom
+Text Notes 9200 6250 0    60   ~ 12
+ADS1299
+Text Label 7800 6100 2    60   ~ 0
+GND_NISO
 $EndSCHEMATC
