File: Desarrollo/Hardware/PonchoERG.kicad_pcb (KiCad board)
At the start: 2 copper layers, 85.9 x 80.5 mm, 108 parts, among them J1 Entradas Analógicas, J2 IOs Multipropósito, U1 TPD2E001, U10 ADS1299, U11 ADuM6401, U12 ADuM2401, U13 NCP1117ST33T3G, U14 OPA2376, U15 TPD2E001, U2 TPD2E001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

Commit message: Actualización final. Serigrafía nueva de jumpers y logos que se habían borrado de PONCHO y OPEN HARDWARE. PLACA TERMINADA.
Parts:
- removed MP?: Plantilla_EDU-CIAA, Poncho_Esqueleto:Plantilla_EDU-CIAA
- added G***: LOGO, Poncho_Esqueleto:Logo_Poncho, F.Cu at (123.5, 73.5)
- added G101: Logo_OSHWA, Poncho_Esqueleto:Logo_OSHWA, F.Cu at (123.5, 144.0)
- added Jumper_Config1: J_CFG, footprints:Jumpers_Default, F.Cu at (125.2, 135.4)
- added Slot_1: Fiducial, Fiducials:Fiducial_1mm_Dia_2.54mm_Outer_CopperTop, F.Cu at (123.5, 121.0)
- added Slot_2: Slot_2, Fiducials:Fiducial_1mm_Dia_2.54mm_Outer_CopperTop, F.Cu at (123.4, 92.6)
- moved FD3 28.0 mm to (108.0, 143.0)
- moved FD7 28.0 mm to (108.0, 143.0)
- moved FD1 27.0 mm to (109.0, 74.0)
- moved FD5 27.0 mm to (109.0, 74.0)
- moved FD2 1.12 mm to (171.0, 73.0)
- moved FD6 1.12 mm to (171.0, 73.0)
- moved MH3 0.71 mm to (104.0, 71.5)
- moved MH4 0.50 mm to (104.0, 144.5)
- moved MH1 0.25 mm to (182.2, 71.5)
- moved MH2 0.25 mm to (182.2, 144.5)
Routing:
- net GNDA: track 523.2 -> 656.0 mm, vias 97 -> 89
- net /AISLACIÓN/GND_NISO: track 309.0 -> 295.4 mm, vias 71 -> 36
- net Net-(J1-Pad1): track 28.4 -> 27.0 mm
Other:
- net class Default: trace_width 0.1 -> 0.2
- rule trace_min: 0.1 -> 0.2
- board text added: "1+"
- board text added: "1-"
- board text added: "2+"
- board text added: "2-"
- board text added: "3+"
- board text added: "3-"
- board text added: "4+"
- board text added: "4-"
- board text added: "5+"
- board text added: "5-"
- board text added: "6+"
- board text added: "6-"
- board text added: "7+"
- board text added: "7-"
- board text added: "8+"
- board text added: "8-"
- board text added: "BIAS_SHD"
- board text added: "Default"
- board text added: "J2"
- board text added: "JP1"
- board text added: "JP2"
- board text added: "JP3"
- board text added: "JP4"
- board text removed: "1+ 1- 2+ 2- 3+ 3- 4+ 4- 5+ 5- 6+ 6- 7+ 7- 8+ 8- IN_REF BIAS_DRV BIAS_ELEC BIAS_SHD"
- board text removed: "BUFFER"
- board text removed: "Buffer_IN"
- board text removed: "GPIO_4"
- board text removed: "IN_REF_Buffer"
- board text removed: "OFF"
- board text removed: "ON"
- board text removed: "SHIELD"
- board text removed: "SRB1"
- board text removed: "SRB2"
